File: mfos_vco.sch (EAGLE design)
At the start: 60 parts, among them IC1 TL072P, IC2 TL072P, IC3 TL072P, T1 2N3904, T2 2N3904, U1 POWER, U2 2N5457

Commit message: ready to try lm394
Parts:
- removed T1, T2: 2N3904, transistor:2N3904
- added IC4: LM394N, synthdiy:LM394N
- added JP1: (no value), SparkFun-Connectors:M05LOCK_LONGPADS
- renumbered R14 to HIGH_FREQ_TRIM, R2 to SCALE_ADJ
Connections:
- net +12V: now also JP1.3
- net -12V: now also JP1.1
- net GND: now also IC4.B1, JP1.2; no longer T1.B
- net N$12: now also IC4.E1, IC4.E2; no longer T1.E, T2.E
- net N$13: now also IC4.C2; no longer T2.C
- net N$23: now also IC4.C1; no longer T1.C
- net N$33: now also JP1.4
- net N$35: now also JP1.5
- net N$8: now also IC4.B2; no longer T2.B
Other:
- moved on the sheet: IC1B
